File: IO_BOARD.kicad_pcb (KiCad board)
At the start: 4 copper layers, 18 x 23.5 mm, 6 parts, among them J2 TYPE-C-31-M-12

Commit message: Fix HRO TYPE-C-31-M-12 land pattern
Parts:
- moved J2 4.52 mm to (9.00, 4.77)
Changed lines of the file:
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@@
   (pad "32" thru_hole roundrect (at 1.33 1.59 0) (size 2.60 1.50) (drill 0.85 (offset -0.50 0)) (layers "*.Cu" "*.Mask") (remove_unused_layers no) (roundrect_rratio 0) (chamfer_ratio 0.2) (chamfer top_left top_right bottom_left bottom_right) (net 23 "VSYS"))
  )
-(footprint "TYPE-C-31-M-12" (layer "F.Cu") (at 9.0 0.25)
-  (fp_text reference "J2" (at 0 3.9) (layer "F.SilkS") (effects (font (size 0.5 0.5) (thickness 0.08))))
-  (fp_text value "TYPE-C-31-M-12" (at 0 5.0) (layer "F.Fab") hide (effects (font (size 1 1) (thickness 0.15))))
-  (fp_rect (start -4.47 -0.20) (end 4.47 7.15) (stroke (width 0.10) (type default)) (fill none) (layer "F.SilkS"))
-  (fp_text user "USB-C" (at 0 5.8) (layer "F.SilkS") (effects (font (size 0.6 0.6) (thickness 0.1))))
-  (pad "A1" smd rect (at -3.25 3.05) (size 0.60 1.30) (layers "F.Cu" "F.Paste" "F.Mask") (net 22 "GND"))
-  (pad "A4" smd rect (at -2.45 3.05) (size 0.60 1.30) (layers "F.Cu" "F.Paste" "F.Mask") (net 24 "USB_VBUS"))
-  (pad "A5" smd rect (at -1.25 3.05) (size 0.30 1.30) (layers "F.Cu" "F.Paste" "F.Mask"))
-  (pad "A6" smd rect (at -0.25 3.05) (size 0.30 1.30) (layers "F.Cu" "F.Paste" "F.Mask") (net 26 "USB_D+"))
-  (pad "A7" smd rect (at 0.25 3.05) (size 0.30 1.30) (layers "F.Cu" "F.Paste" "F.Mask") (net 25 "USB_D-"))
-  (pad "A8" smd rect (at 1.25 3.05) (size 0.30 1.30) (layers "F.Cu" "F.Paste" "F.Mask"))
-  (pad "A9" smd rect (at 2.45 3.05) (size 0.60 1.30) (layers "F.Cu" "F.Paste" "F.Mask") (net 24 "USB_VBUS"))
-  (pad "A12" smd rect (at 3.25 3.05) (size 0.60 1.30) (layers "F.Cu" "F.Paste" "F.Mask") (net 22 "GND"))
-  (pad "B1" smd rect (at 3.25 3.05) (size 0.60 1.30) (layers "F.Cu" "F.Paste" "F.Mask") (net 22 "GND"))
-  (pad "B4" smd rect (at 2.45 3.05) (size 0.60 1.30) (layers "F.Cu" "F.Paste" "F.Mask") (net 24 "USB_VBUS"))
-  (pad "B5" smd rect (at 1.75 3.05) (size 0.30 1.30) (layers "F.Cu" "F.Paste" "F.Mask"))
-  (pad "B6" smd rect (at 0.75 3.05) (size 0.30 1.30) (layers "F.Cu" "F.Paste" "F.Mask") (net 26 "USB_D+"))
-  (pad "B7" smd rect (at -0.75 3.05) (size 0.30 1.30) (layers "F.Cu" "F.Paste" "F.Mask") (net 25 "USB_D-"))
-  (pad "B8" smd rect (at -1.75 3.05) (size 0.30 1.30) (layers "F.Cu" "F.Paste" "F.Mask"))
-  (pad "B9" smd rect (at -2.45 3.05) (size 0.60 1.30) (layers "F.Cu" "F.Paste" "F.Mask") (net 24 "USB_VBUS"))
-  (pad "B12" smd rect (at -3.25 3.05) (size 0.60 1.30) (layers "F.Cu" "F.Paste" "F.Mask") (net 22 "GND"))
-  (pad "S1" thru_hole oval (at -3.95 1.55) (size 1.20 2.00) (drill 0.80) (layers "*.Cu" "*.Mask"))
-  (pad "S2" thru_hole oval (at 3.95 1.55) (size 1.20 2.00) (drill 0.80) (layers "*.Cu" "*.Mask"))
-  (pad "S3" thru_hole oval (at -3.95 3.00) (size 1.20 1.80) (drill 0.80) (layers "*.Cu" "*.Mask"))
-  (pad "S4" thru_hole oval (at 3.95 3.00) (size 1.20 1.80) (drill 0.80) (layers "*.Cu" "*.Mask"))
- )
- (footprint "FH40-24S-0.5SV" (layer "F.Cu") (at 9 10.0)
+(footprint "TYPE-C-31-M-12" (layer "F.Cu") (at 9.0 4.77)
+  (fp_text reference "J2" (at 0 -5.645) (layer "F.SilkS") (effects (font (size 0.5 0.5) (thickness 0.08))))
+  (fp_text value "TYPE-C-31-M-12" (at 0 5.1) (layer "F.Fab") hide (effects (font (size 1 1) (thickness 0.15))))
+  (fp_line (start -4.7 2) (end -4.7 3.9) (stroke (width 0.12) (type default)) (layer "F.SilkS"))
+  (fp_line (start -4.7 -1.9) (end -4.7 0.1) (stroke (width 0.12) (type default)) (layer "F.SilkS"))
+  (fp_line (start 4.7 2) (end 4.7 3.9) (stroke (width 0.12) (type default)) (layer "F.SilkS"))
+  (fp_line (start 4.7 -1.9) (end 4.7 0.1) (stroke (width 0.12) (type default)) (layer "F.SilkS"))
+  (fp_line (start -4.7 3.9) (end 4.7 3.9) (stroke (width 0.12) (type default)) (layer "F.SilkS"))
+  (fp_rect (start -5.32 -5.27) (end 5.32 4.15) (stroke (width 0.05) (type default)) (fill none) (layer "F.CrtYd"))
+  (pad "S1" thru_hole oval (at 4.32 1.05) (size 1 1.6) (drill oval 0.6 1.2) (layers "*.Cu" "*.Mask"))
+  (pad "" np_thru_hole circle (at 2.89 -2.6) (size 0.65 0.65) (drill 0.65) (layers "*.Cu" "*.Mask"))
+  (pad "S1" thru_hole oval (at -4.32 1.05) (size 1 1.6) (drill oval 0.6 1.2) (layers "*.Cu" "*.Mask"))
+  (pad "" np_thru_hole circle (at -2.89 -2.6) (size 0.65 0.65) (drill 0.65) (layers "*.Cu" "*.Mask"))
+  (pad "S1" thru_hole oval (at -4.32 -3.13) (size 1 2.1) (drill oval 0.6 1.7) (layers "*.Cu" "*.Mask"))
+  (pad "S1" thru_hole oval (at 4.32 -3.13) (size 1 2.1) (drill oval 0.6 1.7) (layers "*.Cu" "*.Mask"))
+  (pad "A6" smd rect (at -0.25 -4.045) (size 0.3 1.45) (layers "F.Cu" "F.Paste" "F.Mask") (net 26 "USB_D+"))
+  (pad "B5" smd rect (at 1.75 -4.045) (size 0.3 1.45) (layers "F.Cu" "F.Paste" "F.Mask"))
+  (pad "A8" smd rect (at 1.25 -4.045) (size 0.3 1.45) (layers "F.Cu" "F.Paste" "F.Mask"))
+  (pad "B6" smd rect (at 0.75 -4.045) (size 0.3 1.45) (layers "F.Cu" "F.Paste" "F.Mask") (net 26 "USB_D+"))
+  (pad "A7" smd rect (at 0.25 -4.045) (size 0.3 1.45) (layers "F.Cu" "F.Paste" "F.Mask") (net 25 "USB_D-"))
+  (pad "B7" smd rect (at -0.75 -4.045) (size 0.3 1.45) (layers "F.Cu" "F.Paste" "F.Mask") (net 25 "USB_D-"))
+  (pad "A5" smd rect (at -1.25 -4.045) (size 0.3 1.45) (layers "F.Cu" "F.Paste" "F.Mask"))
+  (pad "B8" smd rect (at -1.75 -4.045) (size 0.3 1.45) (layers "F.Cu" "F.Paste" "F.Mask"))
+  (pad "A12" smd rect (at 3.25 -4.045) (size 0.6 1.45) (layers "F.Cu" "F.Paste" "F.Mask") (net 22 "GND"))
+  (pad "B4" smd rect (at 2.45 -4.045) (size 0.6 1.45) (layers "F.Cu" "F.Paste" "F.Mask") (net 24 "USB_VBUS"))
+  (pad "A4" smd rect (at -2.45 -4.045) (size 0.6 1.45) (layers "F.Cu" "F.Paste" "F.Mask") (net 24 "USB_VBUS"))
+  (pad "A1" smd rect (at -3.25 -4.045) (size 0.6 1.45) (layers "F.Cu" "F.Paste" "F.Mask") (net 22 "GND"))
+  (pad "B12" smd rect (at -3.25 -4.045) (size 0.6 1.45) (layers "F.Cu" "F.Paste" "F.Mask") (net 22 "GND"))
+  (pad "B9" smd rect (at -2.45 -4.045) (size 0.6 1.45) (layers "F.Cu" "F.Paste" "F.Mask") (net 24 "USB_VBUS"))
+  (pad "A9" smd rect (at 2.45 -4.045) (size 0.6 1.45) (layers "F.Cu" "F.Paste" "F.Mask") (net 24 "USB_VBUS"))
+  (pad "B1" smd rect (at 3.25 -4.045) (size 0.6 1.45) (layers "F.Cu" "F.Paste" "F.Mask") (net 22 "GND"))
+)
+(footprint "FH40-24S-0.5SV" (layer "F.Cu") (at 9 10.0)
   (fp_text reference "JFFC_VERT" (at 0 -3.8) (layer "F.SilkS")
     (effects (font (size 0.45 0.45) (thickness 0.08)))
